File: Hardware/BLDC ESC/BLDC ESC.kicad_pcb (KiCad board)
At the start: 2 copper layers, 146.2 x 72.2 mm, 73 parts, among them J1 Motor Terminal, J2 Power Input, J3 DIRECTION SELECT, J4 PWM SELECT, J5 UART Debug Port, J6 ISP Port, J7 PWM INPUT, Q1 IRF1405, Q2 IRF1405, Q3 IRF1405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

Commit message: PCB errors corrected
Parts:
- J3: value DIRECTION SELECT -> DIR SEL
- J4: value PWM SELECT -> PWM SEL
- J7: value PWM INPUT -> PWM
Routing:
- net /PH_C_MOT: track 107.7 -> 172.3 mm
- net /PH_B_MOT: track 121.0 -> 173.1 mm
- net /PH_A_MOT: track 148.2 -> 199.8 mm
- net Net-(D3-K): track 5.86 -> 13.0 mm
- net Net-(D2-K): track 5.80 -> 12.6 mm
- net Net-(D1-K): track 6.34 -> 12.9 mm
- net +12V: track 183.6 -> 181.6 mm
- net Net-(U2-LO): track 28.9 -> 28.3 mm
- net Net-(U3-LO): track 29.3 -> 28.8 mm
